File: dilemma/dilemma.kicad_pcb (KiCad board)
At the start: 2 copper layers, 134 x 107.4 mm, 83 parts, among them J1 S3B-PH-SM4-TB(LF)(SN), J2 Serial, J3 BATTERY_CONN_DEANS, J5 S3B-PH-SM4-TB(LF)(SN), SW1 SW_Push, SW10 SW_Push, SW11 SW_Push, SW12 SW_Push, SW13 SW_Push, SW14 SW_Push, SW15 SW_Push, SW16 SW_Push, SW17 locked, SW18 SW_Push, SW2 SW_Push, SW26 SW_SPST, SW3 SW_Push, SW37 SW_SPST, SW4 SW_Push, SW5 SW_Push, SW6 SW_Push, SW7 SW_Push, SW8 SW_Push, SW9 SW_Push, U2 eliteC

Commit message: mostly step and organization
Parts:
- added H2: M4, local-libraries:MountingHole_3mm_Pad_thin, F.Cu at (208.6, 114.8)
