File: dilemma_assembled/dilemma.kicad_sch (KiCad schematic)
At the start: 105 parts, among them J1 USB_C_Receptacle_USB2.0, J101 trackball, J102 Serial, J103 Serial, J104 Conn_01x02_Female, J107 Conn_01x08_Female, J108 Conn_01x01_Female, J109 Conn_01x01_Female, J113 Cirque, J5 Conn_01x02, SW1 SW_Push, SW101 SW_Push, SW102 SW_Push, SW103 SW_Push, SW104 SW_Push, SW105 SW_Push, SW106 SW_Push, SW107 SW_Push, SW108 SW_Push, SW109 SW_Push, SW110 SW_SPST, SW111 SW_SPST, SW112 SW_Push, SW113 SW_Push, SW114 SW_Push, SW115 SW_Push, SW116 SW_Push, SW117 SW_Push, SW118 SW_Push, SW119 SW_Push, SW2 SW_Push, U1 RP2040, U2 GD25Q80CEIGR, U3 XC6210B332MR-G, Y1 Crystal_GND24

Commit message: pull from main branch
Parts:
- removed H103: M4, local-libraries:MountingHole_3mm_Pad_thin, symbol Mechanical:MountingHole_Pad
- removed J101: trackball, Library:6_PinHeader, symbol Connector:Conn_01x06_Female
- removed J104: Conn_01x02_Female, local-libraries:PinHeader_1x02_P2.54mm_Vertical, symbol Connector:Conn_01x02_Female
- added J105: Conn_01x04_Female, local-libraries:PinHeader_1x04_P2.54mm_Vertical_debug, symbol Connector:Conn_01x04_Female
Connections:
- net +3V3: now also J105.1 (Pin_1)
- net GND: now also R4.1, R5.1, J105.4 (Pin_4); no longer R4.2, R5.2
- net SWCLK: now reaches U1.24 (SWCLK)
- net SWCLK: now also J105.2 (Pin_2)
- net SWD: now reaches U1.25 (SWD)
- net SWD: now also J105.3 (Pin_3)
- net at J1.A5 (CC1): now also R4.2; no longer R4.1
- net at J1.B5 (CC2): now also R5.2; no longer R5.1
- no-connect marks 22 -> 20
Other:
- note added: "Cirque FPC connector"
- note added: "Debug breakout"
- note added: "GPIO breakout"
- note added: "I2C breakout"
- note added: "OLED connector"
- note added: "Reset button"
- note removed: "MCU Left"
- note removed: "OLED Left"
- note removed: "Power"
- note removed: "Pull ups for trackpad"
- note removed: "Reset button Left"
- moved on the sheet: D101, D102, D103, D104, D105, D106, D107, D108, D109, D110, D111, D112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
